File: kicad/cycloadc/cyclo-adc.kicad_pcb (KiCad board)
At the start: 2 copper layers, 85 x 39.5 mm, 12 parts, among them P1 CONN_8, P2 CONN_8, U1 TL431LP

Commit message: misc changes before other changes...
Routing:
- net +AREF: track 266.7 -> 247.9 mm, vias 4 -> 2
- net (no net): track 0.00 -> 2.64 mm
Changed lines of the file:
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@@
   (general
     (links 92)
-    (no_connects 0)
-    (area 115.699999 79.449999 175.800001 118.050001)
+    (no_connects 1)
+    (area 83.786073 78.2215 195.115447 120.07446)
     (thickness 1.6)
     (drawings 56)
-    (tracks 510)
+    (tracks 509)
     (zones 0)
     (modules 12)
@@
   )
   (setup
-    (last_trace_width 0.2)
+    (last_trace_width 0.254)
     (user_trace_width 0.1)
     (user_trace_width 0.2)
@@
     (visible_elements FFFFFF7F)
     (pcbplotparams
-      (layerselection 3178497)
+      (layerselection 271613953)
       (usegerberextensions true)
       (excludeedgelayer true)
@@
       (outputformat 1)
       (mirror false)
-      (drillshape 1)
+      (drillshape 0)
       (scaleselection 1)
-      (outputdirectory ""))
+      (outputdirectory ../gerber/))
   )
   (net 0 "")
@@
       (effects (font (size 1.5 1.5) (thickness 0.15)))
     )
-    (fp_text value CONN_8 (at 0.4 6.8 90) (layer F.SilkS)
+    (fp_text value CONN_8 (at -0.1 -2.9 90) (layer F.SilkS)
       (effects (font (size 1.5 1.5) (thickness 0.15)))
     )
@@
     (effects (font (size 1.5 1.5) (thickness 0.3)))
   )
-  (gr_text "Cyclo-ADC 1.0" (at 136.245 92.41) (layer F.SilkS)
-    (effects (font (size 1.5 1.5) (thickness 0.3)))
-  )
+  (gr_text "Cyclo-ADC 1.0" (at 105.25 99.5 90) (layer F.SilkS)
+    (effects (font (size 1.5 1.5) (thickness 0.3)))
+  )
+  (segment (start 153.35 91.5) (end 153.45 91.4) (width 0.254) (layer B.Cu) (net 0))
+  (segment (start 150.85 91.5) (end 153.35 91.5) (width 0.254) (layer B.Cu) (net 0))
   (segment (start 97.45 106.1) (end 103.15 106.1) (width 0.254) (layer F.Cu) (net 1))
   (segment (start 106.84 102.41) (end 111.25 102.41) (width 0.254) (layer F.Cu) (net 1))
@@
   (via (at 153.69 104.39) (size 0.889) (layers F.Cu B.Cu) (net 1))
   (segment (start 154.75 104) (end 153.69 104.39) (width 0.2) (layer F.Cu) (net 1))
-  (segment (start 157.2 103) (end 155.75 103) (width 0.2) (layer F.Cu) (net 1))
-  (segment (start 155.75 103) (end 154.75 104) (width 0.2) (layer F.Cu) (net 1))
+  (segment (start 157.2 103) (end 155.25 103) (width 0.2) (layer F.Cu) (net 1))
+  (segment (start 155.25 103) (end 154.75 104) (width 0.2) (layer F.Cu) (net 1))
   (segment (start 150.8 94.5) (end 149.25 94.5) (width 0.2) (layer F.Cu) (net 1))
   (segment (start 97.45 101.1) (end 105.95 101.1) (width 0.254) (layer F.Cu) (net 2))
@@
   (segment (start 148.75 95.5) (end 147.75 94.5) (width 0.2) (layer F.Cu) (net 3))
   (segment (start 150.8 95.5) (end 148.75 95.5) (width 0.2) (layer F.Cu) (net 3))
-  (segment (start 157.15 101.5) (end 158.85 101.5) (width 0.2) (layer F.Cu) (net 4) (status 400000))
+  (segment (start 157.15 101.5) (end 158.85 101.5) (width 0.2) (layer F.Cu) (net 4))
   (segment (start 158.35 104) (end 159.35 103) (width 0.2) (layer F.Cu) (net 4))
   (segment (start 159.35 103) (end 159.35 102) (width 0.2) (layer F.Cu) (net 4))
   (via (at 159.35 102) (size 0.889) (layers F.Cu B.Cu) (net 4))
-  (segment (start 158.35 104) (end 157.15 104) (width 0.2) (layer F.Cu) (net 4) (status 800000))
+  (segment (start 158.35 104) (end 157.15 104) (width 0.2) (layer F.Cu) (net 4))
   (segment (start 158.85 101.5) (end 159.35 102) (width 0.2) (layer F.Cu) (net 4))
   (segment (start 118.465 95.331) (end 118.465 96.915) (width 0.254) (layer F.Cu) (net 4))
@@
   (segment (start 162.5 112.25) (end 161.51 113.24) (width 0.2) (layer F.Cu) (net 14))
   (segment (start 161.51 113.24) (end 161.51 114) (width 0.2) (layer F.Cu) (net 14))
+  (segment (start 150.75 102) (end 152.35 102) (width 0.2) (layer F.Cu) (net 15))
+  (segment (start 155.65 104.5) (end 157.15 104.5) (width 0.2) (layer F.Cu) (net 15))
+  (segment (start 155.65 104.8) (end 155.65 104.5) (width 0.2) (layer F.Cu) (net 15))
+  (segment (start 155.15 105.3) (end 155.65 104.8) (width 0.2) (layer F.Cu) (net 15))
+  (segment (start 155.15 106.4) (end 155.15 105.3) (width 0.2) (layer F.Cu) (net 15))
+  (segment (start 154.75 106.8) (end 155.15 106.4) (width 0.2) (layer F.Cu) (net 15))
+  (segment (start 153.55 106.8) (end 154.75 106.8) (width 0.2) (layer F.Cu) (net 15))
+  (segment (start 152.85 106.1) (end 153.55 106.8) (width 0.2) (layer F.Cu) (net 15))
+  (segment (start 152.85 103.8) (end 152.85 106.1) (width 0.2) (layer F.Cu) (net 15))
+  (segment (start 152.45 103.4) (end 152.85 103.8) (width 0.2) (layer F.Cu) (net 15))
+  (segment (start 152.45 102.1) (end 152.45 103.4) (width 0.2) (layer F.Cu) (net 15))
+  (segment (start 152.35 102) (end 152.45 102.1) (width 0.2) (layer F.Cu) (net 15))
   (segment (start 111.25 89.71) (end 106.94 89.71) (width 0.254) (layer F.Cu) (net 15))
   (segment (start 106.94 89.71) (end 98.33 81.1) (width 0.254) (layer F.Cu) (net 15))
@@
   (segment (start 154 94.25) (end 155.25 95.5) (width 0.2) (layer F.Cu) (net 15))
   (segment (start 150.8 93) (end 153.75 93) (width 0.2) (layer F.Cu) (net 15))
-  (segment (start 152.25 102) (end 152.5 102.25) (width 0.2) (layer F.Cu) (net 15))
-  (segment (start 150.8 102) (end 152.25 102) (width 0.2) (layer F.Cu) (net 15))
-  (segment (start 152.5 102.25) (end 152.86 105.76) (width 0.2) (layer F.Cu) (net 15))
-  (segment (start 152.86 105.76) (end 153.464042 106.763489) (width 0.2) (layer F.Cu) (net 15))
-  (segment (start 156 104.5) (end 157.2 104.5) (width 0.2) (layer F.Cu) (net 15))
-  (segment (start 154.32 106.8) (end 156 104.5) (width 0.2) (layer F.Cu) (net 15))
-  (segment (start 153.464042 106.763489) (end 154.32 106.8) (width 0.2) (layer F.Cu) (net 15))
-  (segment (start 159.75 104.5) (end 157.2 104.5) (width 0.2) (layer F.Cu) (net 15))
   (segment (start 168.63 92.37) (end 168.63 83.5) (width 0.2) (layer F.Cu) (net 15))
   (segment (start 157.2 95.5) (end 165.5 95.5) (width 0.2) (layer F.Cu) (net 15))
@@
   (segment (start 174.5 116.75) (end 174.5 98.75) (width 0.254) (layer F.Cu) (net 15))
   (segment (start 120.87 114) (end 120.87 115.62) (width 0.254) (layer F.Cu) (net 15))
-  (segment (start 173.5 98.75) (end 170.5 101.75) (width 0.2) (layer F.Cu) (net 15))
-  (via (at 170.5 101.75) (size 0.889) (layers F.Cu B.Cu) (net 15))
-  (segment (start 170.5 101.75) (end 168.75 103.5) (width 0.2) (layer B.Cu) (net 15))
-  (segment (start 168.75 103.5) (end 160.75 103.5) (width 0.2) (layer B.Cu) (net 15))
-  (via (at 160.75 103.5) (size 0.889) (layers F.Cu B.Cu) (net 15))
-  (segment (start 160.75 103.5) (end 159.75 104.5) (width 0.2) (layer F.Cu) (net 15))
-  (segment (start 174.5 98.75) (end 173.5 98.75) (width 0.2) (layer F.Cu) (net 15))
   (segment (start 155.25 95.5) (end 157.2 95.5) (width 0.2) (layer F.Cu) (net 15))
   (segment (start 97.45 116.1) (end 102.64 116.1) (width 0.254) (layer F.Cu) (net 16))
   (segment (start 102.64 116.1) (end 111.25 107.49) (width 0.254) (layer F.Cu) (net 16))
   (segment (start 111.25 107.49) (end 132.54 107.49) (width 0.254) (layer F.Cu) (net 16))
-  (segment (start 156 103.5) (end 154.25 105.7) (width 0.2) (layer F.Cu) (net 16))
+  (segment (start 155.65 103.5) (end 154.25 105.7) (width 0.2) (layer F.Cu) (net 16))
   (segment (start 154.25 105.7) (end 153.85 105.67) (width 0.2) (layer F.Cu) (net 16))
   (via (at 153.85 105.67) (size 0.889) (layers F.Cu B.Cu) (net 16))
   (segment (start 153.85 105.67) (end 141.18 105.25) (width 0.2) (layer B.Cu) (net 16))
-  (segment (start 156 103.5) (end 157.2 103.5) (width 0.2) (layer F.Cu) (net 16))
+  (segment (start 155.65 103.5) (end 157.2 103.5) (width 0.2) (layer F.Cu) (net 16))
   (segment (start 141.18 105.27) (end 141.18 105.25) (width 0.254) (layer B.Cu) (net 16))
   (segment (start 141.15 105.3) (end 141.18 105.27) (width 0.254) (layer B.Cu) (net 16))
