File: kicad/cycloadc/cyclo-adc.sch (KiCad schematic (older format))
At the start: 8 parts, among them U1 TL431LP

Commit message: various changes... pcb files for cyclo-nexus, cyclo-adc.
Parts:
- removed ADS-0, ADS-1: ADS7957, symbol ADS7957
- removed P?: CONN_10, symbol CONN_10
- added ADC-0, ADC-1: ADS7957, symbol ADS7957
- added P1, P2: CONN_8, symbol CONN_8
- IOPINS0: renamed from Left1; value ADCLEFTPINS -> ADC-0-PINS
- IOPINS1: renamed from Right1; value ADCRIGHTPINS -> ADC-1-PINS
- gave numbers to parts that had none: 1
Connections:
- net 5V is gone; now on net 3.3V: R1.1
- net +AREF: now also ADC-0.29 (+VA), ADC-0.5 (+VA), ADC-1.29 (+VA), ADC-1.5 (+VA), P1.1 (P1), P2.1 (P1)
- net 2.5V: now also ADC-0.4 (REFP), ADC-1.4 (REFP)
- net 3.3V: now also ADC-0.36 (+VBD), ADC-1.36 (+VBD), P1.2 (P2), P2.2 (P2)
- net CH0: now also ADC-0.28 (CH0)
- net CH1: now also ADC-0.27 (CH1)
- net CH10: now also ADC-0.16 (CH10)
- net CH11: now also ADC-0.15 (CH11)
- net CH12: now also ADC-0.14 (CH12)
- net CH13: now also ADC-0.13 (CH13)
- net CH14: now also ADC-0.12 (CH14)
- net CH15: now also ADC-0.11 (CH15)
- net CH16: now also ADC-1.28 (CH0)
- net CH17: now also ADC-1.27 (CH1)
- net CH18: now also ADC-1.26 (CH2)
- net CH19: now also ADC-1.25 (CH3)
- net CH2: now also ADC-0.26 (CH2)
- net CH20: now also ADC-1.24 (CH4)
- net CH21: now also ADC-1.23 (CH5)
- net CH22: now also ADC-1.22 (CH7)
- net CH23: now also ADC-1.22 (CH7)
- net CH24: now also ADC-1.18 (CH8)
- net CH25: now also ADC-1.17 (CH9)
- net CH26: now also ADC-1.16 (CH10)
- net CH27: now also ADC-1.15 (CH11)
- net CH28: now also ADC-1.14 (CH12)
- net CH29: now also ADC-1.13 (CH13)
- net CH3: now also ADC-0.25 (CH3)
- net CH30: now also ADC-1.12 (CH14)
- net CH31: now also ADC-1.11 (CH15)
- net CH4: now also ADC-0.24 (CH4)
- net CH5: now also ADC-0.23 (CH5)
- net CH6: now also ADC-0.22 (CH7)
- net CH7: now also ADC-0.22 (CH7)
- net CH8: now also ADC-0.18 (CH8)
- net CH9: now also ADC-0.17 (CH9)
- net DIO0: now also ADC-0.37 (GPIO0)
- net DIO1: now also ADC-0.38 (GPIO1)
- net DIO2: now also ADC-0.1 (GPIO2)
- net DIO3: now also ADC-0.2 (GPIO3)
- net DIO4: now also ADC-1.37 (GPIO0)
- net DIO5: now also ADC-1.38 (GPIO1)
- net DIO6: now also ADC-1.1 (GPIO2)
- net DIO7: now also ADC-1.2 (GPIO3)
- net GND: now also ADC-0.10 (AGND), ADC-0.19 (AGND), ADC-0.20 (AGND), ADC-0.3 (REFM), ADC-0.30 (AGND), ADC-0.35 (BDGND), ADC-0.6 (AGND), ADC-0.9 (AINM), ADC-1.10 (AGND), ADC-1.19 (AGND), ADC-1.20 (AGND), ADC-1.3 (REFM), ADC-1.30 (AGND), ADC-1.35 (BDGND), ADC-1.6 (AGND), ADC-1.9 (AINM), P1.3 (P3), P2.3 (P3)
- net SCLK: now also ADC-0.32 (SCLK), ADC-1.32 (SCLK), P1.6 (P6), P2.6 (P6)
- new net: ADC-1.7 (MXO), ADC-1.8 (AINP)
- new net: ADC-0.7 (MXO), ADC-0.8 (AINP)
- new net CS0: ADC-0.31 (CS), P1.8 (P8), P2.8 (P8)
- new net CS1: ADC-1.31 (CS), P1.7 (P7), P2.7 (P7)
- new net SDI: ADC-0.33 (SDI), ADC-1.33 (SDI), P1.5 (P5), P2.5 (P5)
- new net SDO: ADC-0.34 (SDO), ADC-1.34 (SDO), P1.4 (P4), P2.4 (P4)
Other:
- note added: "screw terminal spacing."
- note removed: "Change to 3.3?\nMight be ok - then allows \nchange of 5V input"
- note removed: "Different names for\nthe same things."
- note removed: "More general purpose: jumper for + and - REFS\n- AGND and +VA, but not REFP and REFM?\n"
Changed lines of the file:
@@
 LIBS:contrib
 LIBS:valves
-LIBS:cyclophone-cache
 LIBS:cyclo-adc-cache
-EELAYER 27 0
+EELAYER 24 0
 EELAYER END
 $Descr User 17000 11000
@@
 GND
 $Comp
-L ADCLEFTPINS Left1
+L ADCLEFTPINS IOPINS0
 U 1 1 53274A2C
 P 7900 7450
-F 0 "Left1" H 7850 5950 60  0000 C CNN
-F 1 "ADCLEFTPINS" H 7900 8450 60  0000 C CNN
+F 0 "IOPINS0" H 7850 5950 60  0000 C CNN
+F 1 "ADC-0-PINS" H 7900 8450 60  0000 C CNN
 F 2 "" H 7900 7450 60  0001 C CNN
 F 3 "" H 7900 7450 60  0001 C CNN
@@
 $EndComp
 $Comp
-L ADCRIGHTPINS Right1
+L ADCRIGHTPINS IOPINS1
 U 1 1 53274980
 P 10800 7450
-F 0 "Right1" H 10750 5950 60  0000 C CNN
-F 1 "ADCRIGHTPINS" H 10800 8450 60  0000 C CNN
+F 0 "IOPINS1" H 10750 5950 60  0000 C CNN
+F 1 "ADC-1-PINS" H 10800 8450 60  0000 C CNN
 F 2 "" H 10800 7450 60  0001 C CNN
 F 3 "" H 10800 7450 60  0001 C CNN
@@
 Text GLabel 6700 4750 0    60   Input ~ 0
 GND
-Text GLabel 13900 5500 2    60   Input ~ 0
+Text GLabel 14550 4350 0    60   Input ~ 0
 CS0
-Text GLabel 13900 5650 2    60   Input ~ 0
-CS1
-Text GLabel 13900 5350 2    60   Input ~ 0
-SCLK
-Text GLabel 13900 5200 2    60   Input ~ 0
-SDI
-Text GLabel 13900 5050 2    60   Input ~ 0
-SDO
-Text GLabel 13650 5500 0    60   Input ~ 0
-CE0
-Text GLabel 13650 5650 0    60   Input ~ 0
-CE1
-Text GLabel 13650 5050 0    60   Input ~ 0
-MOSI
-Text GLabel 13650 5200 0    60   Input ~ 0
-MISO
-Text GLabel 13650 5350 0    60   Input ~ 0
-SCLK
 Text GLabel 9100 2850 2    60   Input ~ 0
 DIO5
@@
 Text GLabel 11750 8550 2    60   Input ~ 0
 CH31
-$Comp
-L ADS7957 ADS-1
-U 1 1 5313C81B
-P 7800 3900
-F 0 "ADS-1" H 7500 5100 60  0000 C CNN
-F 1 "ADS7957" H 7800 4000 60  0000 C CNN
-F 2 "" H 7800 3900 60  0001 C CNN
-F 3 "" H 7800 3900 60  0001 C CNN
-	1    7800 3900
-	1    0    0    -1
-$EndComp
-$Comp
-L ADS7957 ADS-0
-U 1 1 5313C810
-P 3900 3900
-F 0 "ADS-0" H 3600 5100 60  0000 C CNN
-F 1 "ADS7957" H 3900 4000 60  0000 C CNN
-F 2 "" H 3900 3900 60  0001 C CNN
-F 3 "" H 3900 3900 60  0001 C CNN
-	1    3900 3900
-	1    0    0    -1
-$EndComp
 Text GLabel 8750 3250 2    60   Input ~ 0
 SDO
@@
 Text GLabel 14200 3850 0    60   Input ~ 0
 GND
-Text GLabel 14500 4150 0    60   Input ~ 0
-SCLK
-Text GLabel 14200 4050 0    60   Input ~ 0
-MISO
-Text GLabel 14500 3950 0    60   Input ~ 0
-MOSI
-Text GLabel 14450 4350 0    60   Input ~ 0
-CE1
-Text GLabel 14200 4250 0    60   Input ~ 0
-CE0
-Text GLabel 14200 3650 0    60   Input ~ 0
-5V
-Text Notes 13400 4700 0    60   ~ 0
-Different names for\nthe same things.
 Text Notes 9050 5950 0    60   ~ 0
 Identical pinouts for both.  \nShould face opposite directions on layout,\n to allow using two of the same daughtercard, \none for each set of pins.\n
@@
 	0    -1   -1   0
 $EndComp
-Text GLabel 10100 4600 0    60   Input ~ 0
-5V
 $Comp
 L R R1
@@
 Text GLabel 11300 4100 1    60   Input ~ 0
 2.5V
-$Comp
-L GND #PWR1
-U 1 1 534472D8
-P 12000 4700
-F 0 "#PWR1" H 12000 4700 30  0001 C CNN
-F 1 "GND" H 12000 4630 30  0001 C CNN
-F 2 "" H 12000 4700 60  0000 C CNN
-F 3 "" H 12000 4700 60  0000 C CNN
-	1    12000 4700
-	1    0    0    -1
-$EndComp
 Wire Wire Line
 	11250 8650 12000 8650
@@
 Wire Wire Line
 	6800 4750 6700 4750
-Wire Wire Line
-	13900 5650 13650 5650
-Wire Wire Line
-	13900 5350 13650 5350
-Wire Wire Line
-	13650 5050 13900 5050
 Wire Wire Line
 	3000 2850 2600 2850
@@
 	4800 2850 5150 2850
 Wire Wire Line
-	13650 5200 13900 5200
-Wire Wire Line
-	13650 5500 13900 5500
+	14650 4350 14550 4350
 Wire Wire Line
 	8800 4750 8900 4750
@@
 Wire Wire Line
 	8350 8650 9100 8650
-Wire Wire Line
-	14650 3950 14500 3950
-Wire Wire Line
-	14650 4150 14500 4150
-Wire Wire Line
-	14650 4050 14200 4050
-Wire Wire Line
-	14450 4350 14650 4350
-Wire Wire Line
-	14650 4250 14200 4250
 Wire Wire Line
 	14650 3850 14200 3850
@@
 Added re Dan
 $Comp
-L C C?
+L C C1
 U 1 1 53449C6F
 P 12350 4400
-F 0 "C?" H 12350 4500 40  0000 L CNN
+F 0 "C1" H 12350 4500 40  0000 L CNN
 F 1 "C" H 12356 4315 40  0000 L CNN
 F 2 "~" H 12388 4250 30  0000 C CNN
@@
 Connection ~ 11300 4200
 Connection ~ 12000 4600
-Text Notes 11850 4900 0    60   ~ 0
+Text Notes 12250 4750 0    60   ~ 0
 could leave cap empty
-Text Notes 12850 2800 0    60   ~ 0
-More general purpose:  jumper for + and - REFS\n- AGND and +VA, but not REFP and REFM?\n
-Text Notes 9700 4850 0    60   ~ 0
-Change to 3.3?\nMight be ok - then allows \nchange of 5V input
-$Comp
-L CONN_10 P?
-U 1 1 534AB35E
-P 15000 3900
-F 0 "P?" V 14950 3900 60  0000 C CNN
-F 1 "CONN_10" V 15050 3900 60  0000 C CNN
-F 2 "" H 15000 3900 60  0000 C CNN
-F 3 "" H 15000 3900 60  0000 C CNN
-	1    15000 3900
-	1    0    0    -1
-$EndComp
-Text GLabel 14400 3550 0    60   Input ~ 0
-5V
-Wire Wire Line
-	14650 3550 14400 3550
-Text GLabel 14200 3450 0    60   Input ~ 0
-AREF
-Wire Wire Line
-	14200 3450 14650 3450
+Text GLabel 14200 3650 0    60   Input ~ 0
++AREF
 Text Notes 13200 3250 0    60   ~ 0
 normally jumper pins 1 and 2 for 0 to 5v range.
@@
 Wire Wire Line
 	2700 3150 3000 3150
+Text GLabel 14600 3950 0    60   Input ~ 0
+SDO
+Text GLabel 14300 4050 0    60   Input ~ 0
+SDI
+Text GLabel 14600 4150 0    60   Input ~ 0
+SCLK
+Text GLabel 14300 4250 0    60   Input ~ 0
+CS1
+Wire Wire Line
+	14600 4150 14650 4150
+Wire Wire Line
+	14650 3950 14600 3950
+Wire Wire Line
+	14650 4050 14300 4050
+Wire Wire Line
+	14650 4250 14300 4250
+Text GLabel 10100 4600 0    60   Input ~ 0
+3.3V
+$Comp
+L ADS7957 ADC-1
+U 1 1 535ECD4B
+P 7800 3900
+F 0 "ADC-1" H 7500 5100 60  0000 C CNN
+F 1 "ADS7957" H 7800 4000 60  0000 C CNN
+F 2 "" H 7800 3900 60  0000 C CNN
+F 3 "" H 7800 3900 60  0000 C CNN
+	1    7800 3900
+	1    0    0    -1
+$EndComp
+$Comp
+L ADS7957 ADC-0
+U 1 1 535ECE01
+P 3900 3900
+F 0 "ADC-0" H 3600 5100 60  0000 C CNN
+F 1 "ADS7957" H 3900 4000 60  0000 C CNN
+F 2 "" H 3900 3900 60  0000 C CNN
+F 3 "" H 3900 3900 60  0000 C CNN
+	1    3900 3900
+	1    0    0    -1
+$EndComp
+$Comp
+L CONN_8 P1
+U 1 1 53600A1D
+P 15000 4000
+F 0 "P1" V 14950 4000 60  0000 C CNN
+F 1 "CONN_8" V 15050 4000 60  0000 C CNN
+F 2 "" H 15000 4000 60  0000 C CNN
+F 3 "" H 15000 4000 60  0000 C CNN
+	1    15000 4000
+	1    0    0    -1
+$EndComp
+Text GLabel 14550 5600 0    60   Input ~ 0
+CS0
+Text GLabel 14500 5000 0    60   Input ~ 0
+3.3V
+Text GLabel 14200 5100 0    60   Input ~ 0
+GND
+Wire Wire Line
+	14650 5600 14550 5600
+Wire Wire Line
+	14650 5100 14200 5100
+Wire Wire Line
+	14500 5000 14650 5000
+Wire Wire Line
+	14650 4900 14200 4900
+Text GLabel 14200 4900 0    60   Input ~ 0
++AREF
+Text GLabel 14600 5200 0    60   Input ~ 0
+SDO
+Text GLabel 14300 5300 0    60   Input ~ 0
+SDI
+Text GLabel 14600 5400 0    60   Input ~ 0
+SCLK
+Text GLabel 14300 5500 0    60   Input ~ 0
+CS1
+Wire Wire Line
+	14600 5400 14650 5400
+Wire Wire Line
+	14650 5200 14600 5200
+Wire Wire Line
+	14650 5300 14300 5300
+Wire Wire Line
+	14650 5500 14300 5500
+$Comp
+L CONN_8 P2
+U 1 1 53600AFF
+P 15000 5250
+F 0 "P2" V 14950 5250 60  0000 C CNN
+F 1 "CONN_8" V 15050 5250 60  0000 C CNN
+F 2 "" H 15000 5250 60  0000 C CNN
+F 3 "" H 15000 5250 60  0000 C CNN
+	1    15000 5250
+	1    0    0    -1
+$EndComp
+Text Notes 14050 4650 0    60   ~ 0
+screw terminal spacing.
+Text GLabel 12000 4700 3    60   Input ~ 0
+GND
 $EndSCHEMATC
