File: kicad/cycloadc/cyclo-adc2.kicad_pcb (KiCad board)
At the start: 2 copper layers, 86.5 x 60.8 mm, 16 parts, among them P1 CONN_8, P2 CONN_8, U1 TL431LP

Commit message: a few more tweaks.
Parts:
- moved C2 18.6 mm to (161.1, 107.5), turned to 90 degrees
- moved MH 14.7 mm to (99.8, 139.7)
- moved MH 14.5 mm to (100.0, 89.9)
- moved MH 0.68 mm to (175.2, 105.6)
Routing:
- net +AREF: track 228.8 -> 223.0 mm
- net REFP: track 65.2 -> 63.3 mm
- net GND: track 62.9 -> 61.2 mm, vias 12 -> 13
- net DIO4: track 37.5 -> 38.8 mm
Other:
- net class lowclearance: clearance 0.15 -> 0.1
- board text added: "A25"
- board text added: "A26"
- board text added: "A27"
- board text added: "A28"
- board text added: "CH2"
- board text added: "CH3"
- board text added: "CH4"
- board text removed: "2"
- board text removed: "25"
- board text removed: "26"
- board text removed: "27"
- board text removed: "28"
- board text removed: "3"
- board text removed: "4"

Commit message: last changes before gerbers and ordering.
Other:
- board text added: "Cyclo ADC 1.0"
- board text removed: "Cyclo-ADC 1.0"
