File: kicad/cyclosensor-opamp/cyclosensor-opamp-opamp.kicad_pcb (KiCad board)
At the start: 2 copper layers, 62.2 x 33 mm, 18 parts, among them J1 RJ14, K1 CONN_3, U1 TCRT5000, U2 MCP6001U, U3 MCP6001U

Commit message: pcb design is semi-complete!  looks that way, anyway.
Parts:
- added MH: MountingHole_3mm_RevA_Date21Jun2010, Mounting_Holes:MountingHole_3mm, F.Cu at (170.2, 76.2)
- added MH: MountingHole_3mm_RevA_Date21Jun2010, Mounting_Holes:MountingHole_3mm, F.Cu at (170.2, 99.1)
- moved U3 8.98 mm to (149.9, 80.0)
- moved R5 5.24 mm to (157.5, 80.0), turned to 270 degrees
- moved R1 5.21 mm to (157.6, 85.1)
- moved R9 4.28 mm to (128.0, 96.2), turned to 90 degrees
- moved U1 4.19 mm to (139.7, 87.2)
- moved U2 2.54 mm to (134.6, 78.7)
- moved C1 1.27 mm to (141.0, 74.9)
- moved C2 1.27 mm to (144.8, 74.9)
- moved K1 1.27 mm to (152.4, 74.9)
- moved R8 0.97 mm to (134.2, 74.0), turned to 180 degrees
- moved R7 0.38 mm to (127.0, 74.0), turned to 180 degrees
- turned R6 to 180 degrees
Routing:
- net 5V: track 0.00 -> 118.0 mm, vias 0 -> 2
- net ADC: track 0.00 -> 62.8 mm
- net Net-(GAIN2-Pad1): track 0.00 -> 49.1 mm, vias 0 -> 2
- net lowcut: track 0.00 -> 35.8 mm
- net Net-(R2-Pad1): track 0.00 -> 28.1 mm, vias 0 -> 1
- net Net-(R3-Pad1): track 0.00 -> 26.6 mm, vias 0 -> 2
- net GND: track 0.00 -> 15.5 mm, vias 0 -> 6
- net Net-(R1-Pad1): track 0.00 -> 13.9 mm, vias 0 -> 2
- added copper zone on B.Cu, net GND

Commit message: add mounting holes
Routing:
- net 5V: track 118.0 -> 116.8 mm
Other:
- board text added: "Cyclo Sensor 1.0"

Commit message: misc changes before other changes...
Routing:
- net Net-(R3-Pad1): track 26.6 -> 31.0 mm

Commit message: redo of adc board with thicker traces, caps next to adc chips.
Routing:
- net Net-(R3-Pad1): track 31.0 -> 32.0 mm
- net 5V: track 116.8 -> 117.6 mm
Other:
- net class Thicker added: clearance 0.254, trace_width 1.016, via_dia 0.889, via_drill 0.635
- net class medium added: clearance 0.254, trace_width 0.5, via_dia 0.889, via_drill 0.635
